Commit message: Update README

File: scara_cpe_description/urdf/scara_cpe.xacro (robot description, xacro)
@@ -7,4 +7,5 @@
   <xacro:property name="Base_HEIGHT" value="0.03" />
   <xacro:property name="Link2_HEIGHT" value="-0.025" />
+  <xacro:property name="PI" value="3.14159265359" />
   <xacro:property name="PI_half" value="1.57079632679" />
   <!-- LINK -->
@@ -90,4 +91,5 @@
     <parent link="world"/>
     <child link="camera_link"/>
+    <origin xyz="0 -0.3 0.2" rpy="-${PI_half+0.3} 0 0" />
   </joint>
   <joint name="shoulder_1_joint" type="revolute">

Commit message: bug fix xacro path

File: scara_cpe_description/urdf/scara_cpe.xacro (robot description, xacro)
@@ -1,5 +1,5 @@
 <robot name="scara_cpe" xmlns:xacro="http://ros.org/wiki/xacro" >
   <!-- Import all Gazebo-customization elements, including Gazebo colors -->
-  <xacro:include filename="$(find scara_cpe)/urdf/scara_cpe.gazebo" />
+  <xacro:include filename="$(find scara_cpe_description)/urdf/scara_cpe.gazebo" />
   <xacro:property name="Base_LENGTH" value="0.06" />
   <xacro:property name="Link1_LENGTH" value="0.08" />
@@ -24,5 +24,5 @@
       <origin xyz="0 0.034 0" rpy="-${PI_half} 0 -${PI_half}" />
       <geometry>
-        <mesh filename="package://scara_cpe/urdf/scara_cpe-base_link.dae" scale="0.001 0.001 0.001"/>
+        <mesh filename="package://scara_cpe_description/urdf/scara_cpe-base_link.dae" scale="0.001 0.001 0.001"/>
       </geometry>
     </visual>
@@ -40,5 +40,5 @@
       <origin xyz="0 -0.012 0" rpy="-${PI_half} 0 -${PI_half}" />
       <geometry>
-        <mesh filename="package://scara_cpe/urdf/scara_cpe-link_1.dae" scale="0.001 0.001 0.001"/>
+        <mesh filename="package://scara_cpe_description/urdf/scara_cpe-link_1.dae" scale="0.001 0.001 0.001"/>
       </geometry>
     </visual>
@@ -62,5 +62,5 @@
 	  <origin xyz="0.0133 -0.092 0" rpy="-${PI_half} 0 -1.42579632679" />  <!-- -1.42579632679  - pi/2 + 0.145 -->
       <geometry>
-        <mesh filename="package://scara_cpe/urdf/scara_cpe-link_2.dae" scale="0.001 0.001 0.001"/>
+        <mesh filename="package://scara_cpe_description/urdf/scara_cpe-link_2.dae" scale="0.001 0.001 0.001"/>
       </geometry>
     </visual>
