Commit message: add branch ros2-template

File: scara_cpe_description/urdf/scara_cpe.urdf (robot description, URDF)
Before this commit: robot scara_cpe, 6 links, 5 joints
Links:
- link base_link: geometry collision mesh filename=file:///home/raph/ros2_move_ws/install/scara_cpe_descriptio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 scale=0.001 0.001 0.001; visual mesh filename=file:///home/raph/ros2_move_ws/install/scara_cpe_descriptio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 scale=0.001 0.001 0.001
- link link1: geometry collision box size=0.02 0.04 0.05; visual mesh filename=file:///home/raph/ros2_move_ws/install/scara_cpe_descriptio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 scale=0.001 0.001 0.001
- link link2: geometry collision box size=0.032 0.047 0.06; visual mesh filename=file:///home/raph/ros2_move_ws/install/scara_cpe_descriptio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 scale=0.001 0.001 0.001
Joints:
- joint shoulder_1_joint: limit lower=-1.57079632679 upper=1.57079632679 effort=1.5 velocity=1.0 -> lower=-1.57079632679 upper=1.57079632679 effort=0.1 velocity=1
- joint shoulder_2_joint: limit lower=-2.8 upper=2.8 effort=1.5 velocity=1.0 -> lower=-2.8 upper=2.8 effort=0.1 velocity=1
